File: Hug_Sensing_Plush_wangyj05/esp32.kicad_sch (KiCad schematic)
At the start: 7 parts, among them SW1 SW_SPST, SW2 SW_SPST, U3 ESP32-S3-WROOM-1-N4

Commit message: Updated layout
Connections:
- net SCL_motor: now also U3.25 (IO48); no longer U3.29 (IO36)
- net SCL_sensor: now also U3.30 (IO37); no longer U3.5 (IO5)
- net SDA_motor: now also U3.24 (IO47); no longer U3.30 (IO37)
- net SDA_sensor: now also U3.29 (IO36); no longer U3.4 (IO4)
Changed lines of the file:
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@@
   (no_connect (at 77.47 68.58))
   (no_connect (at 77.47 91.44))
-  (no_connect (at 107.95 106.68))
   (no_connect (at 107.95 88.9))
   (no_connect (at 77.47 93.98))
@@
   (no_connect (at 107.95 96.52))
   (no_connect (at 77.47 99.06))
+  (no_connect (at 77.47 76.2))
   (no_connect (at 107.95 93.98))
   (no_connect (at 77.47 81.28))
+  (no_connect (at 77.47 78.74))
   (no_connect (at 77.47 71.12))
   (no_connect (at 77.47 106.68))
@@
   (no_connect (at 77.47 96.52))
   (no_connect (at 77.47 60.96))
-  (no_connect (at 107.95 104.14))
   (no_connect (at 77.47 73.66))
   (no_connect (at 77.47 86.36))
@@
     (effects (font (size 1.27 1.27)) (justify left bottom))
   )
+  (hierarchical_label "SCL_sensor" (shape input) (at 107.95 83.82 0) (fields_autoplaced)
+    (effects (font (size 1.27 1.27)) (justify left))
+  )
   (hierarchical_label "ESP32_USB_D+" (shape input) (at 107.95 73.66 0) (fields_autoplaced)
     (effects (font (size 1.27 1.27)) (justify left))
@@
     (effects (font (size 1.27 1.27)) (justify left))
   )
-  (hierarchical_label "SDA_motor" (shape input) (at 107.95 83.82 0) (fields_autoplaced)
+  (hierarchical_label "SCL_motor" (shape input) (at 107.95 106.68 0) (fields_autoplaced)
     (effects (font (size 1.27 1.27)) (justify left))
   )
-  (hierarchical_label "SCL_motor" (shape input) (at 107.95 81.28 0) (fields_autoplaced)
+  (hierarchical_label "SDA_sensor" (shape input) (at 107.95 81.28 0) (fields_autoplaced)
     (effects (font (size 1.27 1.27)) (justify left))
   )
-  (hierarchical_label "SDA_sensor" (shape input) (at 77.47 76.2 180) (fields_autoplaced)
-    (effects (font (size 1.27 1.27)) (justify right))
+  (hierarchical_label "SDA_motor" (shape input) (at 107.95 104.14 0) (fields_autoplaced)
+    (effects (font (size 1.27 1.27)) (justify left))
   )
   (hierarchical_label "3V3" (shape input) (at 113.03 50.8 0) (fields_autoplaced)
     (effects (font (size 1.27 1.27)) (justify left))
   )
-  (hierarchical_label "SCL_sensor" (shape input) (at 77.47 78.74 180) (fields_autoplaced)
-    (effects (font (size 1.27 1.27)) (justify right))
-  )
   (symbol (lib_id "power:GND") (at 114.3 137.16 0) (unit 1)

Commit message: Edited PCB layout
Parts:
- TP6: value TestPoint -> TP: ESP_EN
Changed lines of the file:
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@@
       (effects (font (size 1.27 1.27)) (justify left))
     )
-    (property "Value" "TestPoint" (at 80.01 51.308 0)
+    (property "Value" "TP: ESP_EN" (at 80.01 51.308 0)
       (effects (font (size 1.27 1.27)) (justify left))
     )
