File: Hug_Sensing_Plush_wangyj05/Hug_Sensing_Plush_wangyj05.kicad_sch (KiCad schematic)
At the start: 8 parts

Commit message: Edited board layout
Parts:
- added J3, J4: Wire Pad, Connector_Wire:SolderWirePad_1x01_SMD_1x2mm, symbol Connector:Conn_01x01_Pin
Connections:
- net +5V: now also J3.1 (Pin_1)
- net GND: now also J4.1 (Pin_1)
Changed lines of the file:
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@@
   )
   (text "Leave two pads to connect power receiver to 5V and GND."
-    (at 53.34 29.21 0)
+    (at 55.88 27.94 0)
     (effects (font (size 1.27 1.27)) (justify left bottom))
   )
@@
     )
   )
+  (symbol (lib_id "power:GND") (at 64.77 25.4 0) (unit 1)
+    (in_bom yes) (on_board yes) (dnp no) (fields_autoplaced)
+    (property "Reference" "#PWR037" (at 64.77 31.75 0)
+      (effects (font (size 1.27 1.27)) hide)
+    )
+    (property "Value" "GND" (at 64.77 30.48 0)
+      (effects (font (size 1.27 1.27)))
+    )
+    (property "Footprint" "" (at 64.77 25.4 0)
+      (effects (font (size 1.27 1.27)) hide)
+    )
+    (property "Datasheet" "" (at 64.77 25.4 0)
+      (effects (font (size 1.27 1.27)) hide)
+    )
+    (pin "1")
+    (instances
+      (project "Hug_Sensing_Plush_wangyj05"
+        (path "/352d7abe-fc72-4473-8b68-62eecf44f496"
+          (reference "#PWR037") (unit 1)
+        )
+      )
+    )
+  )
   (symbol (lib_id "power:GND") (at 25.4 158.75 0) (unit 1)
     (in_bom yes) (on_board yes) (dnp no) (fields_autoplaced)
@@
         (path "/352d7abe-fc72-4473-8b68-62eecf44f496"
           (reference "H3") (unit 1)
+        )
+      )
+    )
+  )
+  (symbol (lib_id "Connector:Conn_01x01_Pin") (at 59.69 25.4 0) (unit 1)
+    (in_bom yes) (on_board yes) (dnp no) (fields_autoplaced)
+    (property "Reference" "J4" (at 60.325 20.32 0)
+      (effects (font (size 1.27 1.27)))
+    )
+    (property "Value" "Wire Pad" (at 60.325 22.86 0)
+      (effects (font (size 1.27 1.27)))
+    )
+    (property "Footprint" "Connector_Wire:SolderWirePad_1x01_SMD_1x2mm" (at 59.69 25.4 0)
+      (effects (font (size 1.27 1.27)) hide)
+    )
+    (property "Datasheet" "~" (at 59.69 25.4 0)
+      (effects (font (size 1.27 1.27)) hide)
+    )
+    (pin "1")
+    (instances
+      (project "Hug_Sensing_Plush_wangyj05"
+        (path "/352d7abe-fc72-4473-8b68-62eecf44f496"
+          (reference "J4") (unit 1)
         )
       )
@@
     )
   )
+  (symbol (lib_id "Connector:Conn_01x01_Pin") (at 59.69 21.59 0) (unit 1)
+    (in_bom yes) (on_board yes) (dnp no) (fields_autoplaced)
+    (property "Reference" "J3" (at 60.325 16.51 0)
+      (effects (font (size 1.27 1.27)))
+    )
+    (property "Value" "Wire Pad" (at 60.325 19.05 0)
+      (effects (font (size 1.27 1.27)))
+    )
+    (property "Footprint" "Connector_Wire:SolderWirePad_1x01_SMD_1x2mm" (at 59.69 21.59 0)
+      (effects (font (size 1.27 1.27)) hide)
+    )
+    (property "Datasheet" "~" (at 59.69 21.59 0)
+      (effects (font (size 1.27 1.27)) hide)
+    )
+    (pin "1")
+    (instances
+      (project "Hug_Sensing_Plush_wangyj05"
+        (path "/352d7abe-fc72-4473-8b68-62eecf44f496"
+          (reference "J3") (unit 1)
+        )
+      )
+    )
+  )
   (symbol (lib_id "Device:R_Small") (at 223.52 29.21 0) (unit 1)
     (in_bom yes) (on_board yes) (dnp no) (fields_autoplaced)
@@
         )
       )
+    )
+  )
+  (symbol (lib_id "power:+5V") (at 64.77 21.59 0) (unit 1)
+    (in_bom yes) (on_board yes) (dnp no) (fields_autoplaced)
+    (property "Reference" "#PWR036" (at 64.77 25.4 0)
+      (effects (font (size 1.27 1.27)) hide)
+    )
+    (property "Value" "+5V" (at 64.77 16.51 0)
+      (effects (font (size 1.27 1.27)))
+    )
+    (property "Footprint" "" (at 64.77 21.59 0)
+      (effects (font (size 1.27 1.27)) hide)
+    )
+    (property "Datasheet" "" (at 64.77 21.59 0)
+      (effects (font (size 1.27 1.27)) hide)
+    )
+    (pin "1")
+    (instances
+      (project "Hug_Sensing_Plush_wangyj05"
+        (path "/352d7abe-fc72-4473-8b68-62eecf44f496"
+          (reference "#PWR036") (unit 1)
+        )
+      )

Commit message: Updated layout
Parts:
- J3: value Wire Pad -> Charger Header 5V
- J4: value Wire Pad -> Charger Header GND
Changed lines of the file:
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@@
       (effects (font (size 1.27 1.27)))
     )
-    (property "Value" "Wire Pad" (at 60.325 22.86 0)
+    (property "Value" "Charger Header GND" (at 60.325 22.86 0)
       (effects (font (size 1.27 1.27)))
     )
@@
       (effects (font (size 1.27 1.27)))
     )
-    (property "Value" "Wire Pad" (at 60.325 19.05 0)
+    (property "Value" "Charger Header 5V" (at 60.325 19.05 0)
       (effects (font (size 1.27 1.27)))
     )

Commit message: Updated board layout
Parts:
- added H5: EECS Logo, Project Library:EECSLogo, symbol Mechanical:MountingHole
- added H6: MechELogo, Project Library:MechELogo, symbol Mechanical:MountingHole
- added H7: EdgertonLogo, Project Library:EdgertonLogo, symbol Mechanical:MountingHole
Changed lines of the file:
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@@
+    )
+  )
+  (symbol (lib_id "Mechanical:MountingHole") (at 71.12 185.42 0) (unit 1)
+    (in_bom yes) (on_board yes) (dnp no) (fields_autoplaced)
+    (property "Reference" "H7" (at 73.66 184.15 0)
+      (effects (font (size 1.27 1.27)) (justify left))
+    )
+    (property "Value" "EdgertonLogo" (at 73.66 186.69 0)
+      (effects (font (size 1.27 1.27)) (justify left))
+    )
+    (property "Footprint" "Project Library:EdgertonLogo" (at 71.12 185.42 0)
+      (effects (font (size 1.27 1.27)) hide)
+    )
+    (property "Datasheet" "" (at 71.12 185.42 0)
+      (effects (font (size 1.27 1.27)) hide)
+    )
+    (instances
+      (project "Hug_Sensing_Plush_wangyj05"
+        (path "/352d7abe-fc72-4473-8b68-62eecf44f496"
+          (reference "H7") (unit 1)
+        )
+      )
     )
   )
@@
         )
       )
+    )
+  )
+  (symbol (lib_id "Mechanical:MountingHole") (at 54.61 185.42 0) (unit 1)
+    (in_bom no) (on_board yes) (dnp no) (fields_autoplaced)
+    (property "Reference" "H6" (at 57.15 184.15 0)
+      (effects (font (size 1.27 1.27)) (justify left))
+    )
+    (property "Value" "MechELogo" (at 57.15 186.69 0)
+      (effects (font (size 1.27 1.27)) (justify left))
+    )
+    (property "Footprint" "Project Library:MechELogo" (at 54.61 185.42 0)
+      (effects (font (size 1.27 1.27)) hide)
+    )
+    (property "Datasheet" "" (at 54.61 185.42 0)
+      (effects (font (size 1.27 1.27)) hide)
+    )
+    (instances
+      (project "Hug_Sensing_Plush_wangyj05"
+        (path "/352d7abe-fc72-4473-8b68-62eecf44f496"
+          (reference "H6") (unit 1)
+        )
+      )
+    )
+  )
+  (symbol (lib_id "Mechanical:MountingHole") (at 36.83 185.42 0) (unit 1)
+    (in_bom no) (on_board yes) (dnp no) (fields_autoplaced)
+    (property "Reference" "H5" (at 39.37 184.15 0)
+      (effects (font (size 1.27 1.27)) (justify left))
+    )
+    (property "Value" "EECS Logo" (at 39.37 186.69 0)
+      (effects (font (size 1.27 1.27)) (justify left))
+    )
+    (property "Footprint" "Project Library:EECSLogo" (at 36.83 185.42 0)
+      (effects (font (size 1.27 1.27)) hide)
+    )
+    (property "Datasheet" "" (at 36.83 185.42 0)
+      (effects (font (size 1.27 1.27)) hide)
+    )
+    (instances
+      (project "Hug_Sensing_Plush_wangyj05"
+        (path "/352d7abe-fc72-4473-8b68-62eecf44f496"
+          (reference "H5") (unit 1)
+        )
+      )
